Commit message: separate robot models for base, hand and gripper are added

File: urdf/iai_student_robot_hand.xacro (robot description, xacro)
@@ -7,9 +7,9 @@
         <color rgba="0 0 0.8 1"/>
     </material>
+    <material name="green">
+        <color rgba="0.0 0.8 0.0 1.0"/>
+    </material>
     <material name="grey">
         <color rgba="0.2 0.2 0.2 1.0"/>
-    </material>
-    <material name="green">
-        <color rgba="0.0 1.0 0.0 1.0"/>
     </material>
     <material name="orange">
@@ -28,66 +28,7 @@
     <xacro:property name="pi" value="3.14"/>
     <xacro:property name="chassis_box_height" value="0.07"/>
-    <xacro:property name="platform_cylinder_length" value="0.05"/>
     <xacro:property name="arm_cylinder_length" value="0.18"/>
     <link name="base_link">
-        <!-- chassis box -->
-        <visual>
-            <origin rpy="0 0 0" xyz="0 0 ${chassis_box_height/2 + wheel_radius/2}"/>
-            <geometry>
-                <box size="0.5 0.3 ${chassis_box_height}"/>
-            </geometry>
-            <material name="orange"/>
-        </visual>
     </link>
-    <link name="caster_link">
-    <!-- caster front -->
-        <visual name="caster_front_visual">
-            <origin rpy=" 0 0 0" xyz="0.2 0 0.05"/>
-            <geometry>
-                <sphere radius="0.05"/>
-            </geometry>
-            <material name="green"/>
-        </visual>
-    </link>
-    <joint name="caster_joint" type="fixed">
-        <origin rpy="0 0 0" xyz="0.0 0.0 0"/>
-        <child link="caster_link"/>
-        <parent link="base_link"/>
-        <axis rpy="0 0 0" xyz="0 0 0"/>
-    </joint>
-    <link name="right_wheel_link">
-        <visual>
-            <origin rpy="0 1.5707 1.5707" xyz="0 0 0"/>
-            <geometry>
-                <cylinder length="0.04" radius="${wheel_radius}"/>
-            </geometry>
-            <material name="black"/>
-        </visual>
-    </link>
-    <joint name="right_wheel_joint" type="continuous">
-        <origin rpy="0 0 0" xyz="-0.05 0.15 ${chassis_box_height/2 + wheel_radius/2}"/>
-        <child link="right_wheel_link"/>
-        <parent link="base_link"/>
-        <axis rpy="0 0 0" xyz="0 1 0"/>
-        <limit effort="10000" velocity="10"/>
-        <joint_properties damping="1.0" friction="1.0"/>
-    </joint>
-    <link name="left_wheel_link">
-        <visual>
-            <origin rpy="0 1.5707 1.5707" xyz="0 0 0"/>
-            <geometry>
-                <cylinder length="0.04" radius="${wheel_radius}"/>
-            </geometry>
-            <material name="black"/>
-        </visual>
-    </link>
-    <joint name="left_wheel_joint" type="continuous">
-        <origin rpy="0 0 0" xyz="-0.05 -0.15 ${chassis_box_height/2 + wheel_radius/2}"/>
-        <child link="left_wheel_link"/>
-        <parent link="base_link"/>
-        <axis rpy="0 0 0" xyz="0 1 0"/>
-        <limit effort="10000" velocity="10"/>
-        <joint_properties damping="1.0" friction="1.0"/>
-    </joint>
     <link name="torso_link">
         <visual>
@@ -103,5 +44,5 @@
         <parent link="base_link"/>
         <child link="torso_link"/>
-        <origin rpy="0 0 0" xyz="0.0 0.0 ${chassis_box_height + wheel_radius/2}"/>
+        <origin rpy="0 0 0" xyz="0.0 0.0 0"/>
     </joint>
     <link name="upper_arm_link">
